File: v2/kicad/led-matrix/led-matrix.kicad_sch (KiCad schematic)
At the start: 6 parts, among them J1 Conn_02x03_Input, J2 Conn_02x03_Output, U1 MAX7219

Commit message: fix female header
Parts:
- J1: footprint Connector_PinSocket_2.54mm:PinSocket_2x03_P2.54mm_Horizontal -> led-matrix:PinSocket_2x03_P2.54mm_Horizontal
Changed lines of the file:
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@@
     (property "Reference" "J1" (id 0) (at 38.1 87.1982 0))
     (property "Value" "Conn_02x03_Input" (id 1) (at 38.1 89.5096 0))
-    (property "Footprint" "Connector_PinSocket_2.54mm:PinSocket_2x03_P2.54mm_Horizontal" (id 2) (at 30.48 102.87 0)
+    (property "Footprint" "led-matrix:PinSocket_2x03_P2.54mm_Horizontal" (id 2) (at 30.48 102.87 0)
       (effects (font (size 1.27 1.27)) hide)
     )
@@
     )
     (path "/00000000-0000-0000-0000-000061d0c670"
-      (reference "J1") (unit 1) (value "Conn_02x03_Input") (footprint "Connector_PinSocket_2.54mm:PinSocket_2x03_P2.54mm_Horizontal")
+      (reference "J1") (unit 1) (value "Conn_02x03_Input") (footprint "led-matrix:PinSocket_2x03_P2.54mm_Horizontal")
     )
     (path "/00000000-0000-0000-0000-000061d0dd4c"
