File: v2/kicad/led-matrix/led-matrix.kicad_sch (KiCad schematic)
At the start: 6 parts, among them J1 Conn_02x03_Input, J2 Conn_02x03_Output, U1 MAX7219

Commit message: V2: Update schematic
Connections:
- net D_fwd: now also J1.1 (D_fwd), J2.1 (D_fwd); no longer J1.5 (D_fwd), J2.5 (D_ret)
- net VCC: now also J1.5 (VCC), J2.5 (VCC); no longer J1.1 (Vcc), J2.1 (Vcc)
Changed lines of the file:
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@@
+    (stroke (width 0) (type default) (color 0 0 0 0))
+  )
+  (wire (pts (xy 140.97 63.5) (xy 144.78 63.5))
     (stroke (width 0) (type default) (color 0 0 0 0))
   )
@@
     )
   )
-  (global_label "D_fwd" (shape input) (at 50.8 96.52 0) (fields_autoplaced)
-    (effects (font (size 1.27 1.27)) (justify left))
-    (property "Intersheet References" "${INTERSHEET_REFS}" (id 0) (at 58.5671 96.4406 0)
-      (effects (font (size 1.27 1.27)) (justify left) hide)
-    )
-  )
-  (global_label "D_fwd" (shape input) (at 140.97 63.5 0) (fields_autoplaced)
-    (effects (font (size 1.27 1.27)) (justify left))
-    (property "Intersheet References" "${INTERSHEET_REFS}" (id 0) (at 148.7371 63.4206 0)
-      (effects (font (size 1.27 1.27)) (justify left) hide)
+  (global_label "D_fwd" (shape input) (at 25.4 93.98 180) (fields_autoplaced)
+    (effects (font (size 1.27 1.27)) (justify right))
+    (property "Intersheet References" "${INTERSHEET_REFS}" (id 0) (at 17.6329 94.0594 0)
+      (effects (font (size 1.27 1.27)) (justify right) hide)
+    )
+  )
+  (global_label "D_fwd" (shape input) (at 115.57 60.96 180) (fields_autoplaced)
+    (effects (font (size 1.27 1.27)) (justify right))
+    (property "Intersheet References" "${INTERSHEET_REFS}" (id 0) (at 107.8029 61.0394 0)
+      (effects (font (size 1.27 1.27)) (justify right) hide)
     )
   )
@@
     )
   )
-  (global_label "Vcc" (shape input) (at 25.4 93.98 180) (fields_autoplaced)
-    (effects (font (size 1.27 1.27)) (justify right))
-    (property "Intersheet References" "${INTERSHEET_REFS}" (id 0) (at 19.8101 93.9006 0)
-      (effects (font (size 1.27 1.27)) (justify right) hide)
+  (global_label "Vcc" (shape input) (at 50.8 96.52 0) (fields_autoplaced)
+    (effects (font (size 1.27 1.27)) (justify left))
+    (property "Intersheet References" "${INTERSHEET_REFS}" (id 0) (at 56.3899 96.5994 0)
+      (effects (font (size 1.27 1.27)) (justify left) hide)
     )
   )
@@
     )
   )
-  (global_label "Vcc" (shape input) (at 115.57 60.96 180) (fields_autoplaced)
-    (effects (font (size 1.27 1.27)) (justify right))
-    (property "Intersheet References" "${INTERSHEET_REFS}" (id 0) (at 109.9801 60.8806 0)
-      (effects (font (size 1.27 1.27)) (justify right) hide)
+  (global_label "Vcc" (shape input) (at 144.78 63.5 0) (fields_autoplaced)
+    (effects (font (size 1.27 1.27)) (justify left))
+    (property "Intersheet References" "${INTERSHEET_REFS}" (id 0) (at 150.3699 63.5794 0)
+      (effects (font (size 1.27 1.27)) (justify left) hide)
     )
   )
@@
     (property "Reference" "J1" (id 0) (at 38.1 87.1982 0))
     (property "Value" "Conn_02x03_Input" (id 1) (at 38.1 89.5096 0))
-    (property "Footprint" "Connector_PinSocket_2.54mm:PinSocket_2x03_P2.54mm_Horizontal" (id 2) (at 30.48 96.52 0)
+    (property "Footprint" "Connector_PinSocket_2.54mm:PinSocket_2x03_P2.54mm_Horizontal" (id 2) (at 30.48 102.87 0)
       (effects (font (size 1.27 1.27)) hide)
     )
@@
     (property "Reference" "J2" (id 0) (at 128.27 54.1782 0))
     (property "Value" "Conn_02x03_Output" (id 1) (at 128.27 56.4896 0))
-    (property "Footprint" "Connector_PinHeader_2.54mm:PinHeader_2x03_P2.54mm_Horizontal" (id 2) (at 120.65 63.5 0)
-      (effects (font (size 1.27 1.27)) hide)
-    )
+    (property "Footprint" "Connector_PinHeader_2.54mm:PinHeader_2x03_P2.54mm_Horizontal" (id 2) (at 120.65 69.85 0)
+      (effects (font (size 1.27 1.27)) hide)
+    )

Commit message: Changed footprint to handsoldering and added logo
Parts:
- J1: footprint Connector_PinSocket_2.54mm:PinSocket_2x03_P2.54mm_Horizontal -> led-matrix:PinSocket_2x03_P2.54mm_Horizontal
- U1: footprint Package_SO:SOIC-24W_7.5x15.4mm_P1.27mm -> led-matrix:HandSolder.SOIC-24W_7.5x15.4mm_P1.27mm
Changed lines of the file:
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@@
     (property "Reference" "J1" (id 0) (at 38.1 87.1982 0))
     (property "Value" "Conn_02x03_Input" (id 1) (at 38.1 89.5096 0))
-    (property "Footprint" "Connector_PinSocket_2.54mm:PinSocket_2x03_P2.54mm_Horizontal" (id 2) (at 30.48 102.87 0)
+    (property "Footprint" "led-matrix:PinSocket_2x03_P2.54mm_Horizontal" (id 2) (at 30.48 102.87 0)
       (effects (font (size 1.27 1.27)) hide)
     )
@@
       (effects (font (size 1.27 1.27)) (justify left))
     )
-    (property "Footprint" "Package_SO:SOIC-24W_7.5x15.4mm_P1.27mm" (id 2) (at 50.8 49.53 0)
+    (property "Footprint" "led-matrix:HandSolder.SOIC-24W_7.5x15.4mm_P1.27mm" (id 2) (at 50.8 49.53 0)
       (effects (font (size 1.27 1.27)) hide)
     )
@@
     )
     (path "/00000000-0000-0000-0000-000061d0c670"
-      (reference "J1") (unit 1) (value "Conn_02x03_Input") (footprint "Connector_PinSocket_2.54mm:PinSocket_2x03_P2.54mm_Horizontal")
+      (reference "J1") (unit 1) (value "Conn_02x03_Input") (footprint "led-matrix:PinSocket_2x03_P2.54mm_Horizontal")
     )
     (path "/00000000-0000-0000-0000-000061d0dd4c"
@@
     )
     (path "/82db4006-3899-43e0-b593-d936c945d657"
-      (reference "U1") (unit 1) (value "MAX7219") (footprint "Package_SO:SOIC-24W_7.5x15.4mm_P1.27mm")
+      (reference "U1") (unit 1) (value "MAX7219") (footprint "led-matrix:HandSolder.SOIC-24W_7.5x15.4mm_P1.27mm")
     )
   )
