File: v2/kicad/led-matrix/led-matrix.kicad_pcb (KiCad board)
At the start: 2 copper layers, 38 x 38 mm, 6 parts, among them J1 Conn_02x03_Input, J2 Conn_02x03_Output, U1 MAX7219

Commit message: attempt 2 routing
Parts:
- moved R1 13.8 mm to (127.1, 123.3)
- moved C1 12.1 mm to (127.2, 118.2)
- moved U1 0.89 mm to (116.6, 120.8), turned to 0 degrees
Routing:
- net Dout: track 0.00 -> 50.5 mm, vias 0 -> 1
- net D_fwd: track 0.00 -> 43.5 mm
- net Vcc: track 5.51 -> 46.4 mm, vias 0 -> 1
- net load: track 0.00 -> 39.5 mm
- net column2: track 0.00 -> 35.8 mm, vias 0 -> 1
- net row3: track 0.00 -> 35.1 mm
- net clk: track 0.00 -> 31.8 mm
- net column5: track 0.00 -> 28.6 mm, vias 0 -> 1
- net row8: track 0.00 -> 27.5 mm
- net row2: track 0.00 -> 24.6 mm, vias 0 -> 1
- net column8: track 0.00 -> 22.8 mm, vias 0 -> 1
- net row7: track 0.00 -> 22.2 mm
- net column3: track 0.00 -> 22.0 mm, vias 0 -> 1
- net row1: track 0.00 -> 21.8 mm, vias 0 -> 1
- net Din: track 0.00 -> 20.4 mm
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- added copper zone on B.Cu, net GND
- added copper zone on F.Cu, net GND
